File: Kicad/capteur.kicad_pcb (KiCad board)
At the start: 2 copper layers, 68.7 x 57.3 mm, 25 parts, among them J1 Power, J2 Digital/PWM, J3 Analog, J4 Digital/PWM, U2 LTC1050ACN8, U3 MCP41100

Commit message: small change of pcb and update of readme
Parts:
- R1, R2b1, R3, R5, R7, R8: footprint Resistor_THT:R_Axial_DIN0207_L6.3mm_D2.5mm_P5.08mm_Vertical -> Library_Empreinte:R_Axial_DIN0207_L6.3mm_D2.5mm_P5.08mm_Vertical
- R6: renamed from R4; footprint Resistor_THT:R_Axial_DIN0207_L6.3mm_D2.5mm_P5.08mm_Vertical -> Library_Empreinte:R_Axial_DIN0207_L6.3mm_D2.5mm_P5.08mm_Vertical
- R9: renamed from R6; footprint Resistor_THT:R_Axial_DIN0207_L6.3mm_D2.5mm_P5.08mm_Vertical -> Library_Empreinte:R_Axial_DIN0207_L6.3mm_D2.5mm_P5.08mm_Vertical
Other:
- board size 68.7 x 57.3 mm -> 68.7 x 57.6 mm
Changed lines of the file:
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@@
     (pad_to_mask_clearance 0)
     (aux_axis_origin 100 100)
-    (grid_origin 100 100)
+    (grid_origin 147.05 98.79)
     (pcbplotparams
       (layerselection 0x0000000_fffffffe)
@@
     )
   )
-  (footprint "Resistor_THT:R_Axial_DIN0207_L6.3mm_D2.5mm_P5.08mm_Vertical" (layer "F.Cu")
+  (footprint "Library_Empreinte:R_Axial_DIN0207_L6.3mm_D2.5mm_P5.08mm_Vertical" (layer "F.Cu")
     (at 153.34 87.3798 90)
     (descr "Resistor, Axial_DIN0207 series, Axial, Vertical, pin pitch=5.08mm, 0.25W = 1/4W, length*diameter=6.3*2.5mm^2, http://cdn-reichelt.de/documents/datenblatt/B400/1_4W%23YAG.pdf")
@@
     (property "ki_keywords" "R res resistor")
     (attr through_hole)
-    (fp_text reference "R4" (at 2.54 -2.37 90) (layer "F.SilkS")
-        (effects (font (size 1 1) (thickness 0.15)))
-    )
-    (fp_text value "R" (at 2.54 2.37 90) (layer "F.Fab") hide
-        (effects (font (size 1 1) (thickness 0.15)))
-    )
-    (fp_text user "${REFERENCE}" (at 2.54 -2.37 90) (layer "F.Fab")
+    (fp_text reference "R6" (at 2.54 -2.37 270) (layer "F.SilkS")
+        (effects (font (size 1 1) (thickness 0.15)))
+    )
+    (fp_text value "R" (at 2.54 2.37 270) (layer "F.Fab")
+        (effects (font (size 1 1) (thickness 0.15)))
+    )
+    (fp_text user "${REFERENCE}" (at 2.54 -2.37 270) (layer "F.Fab")
         (effects (font (size 1 1) (thickness 0.15)))
     )
@@
     )
   )
-  (footprint "Resistor_THT:R_Axial_DIN0207_L6.3mm_D2.5mm_P5.08mm_Vertical" (layer "F.Cu")
+  (footprint "Library_Empreinte:R_Axial_DIN0207_L6.3mm_D2.5mm_P5.08mm_Vertical" (layer "F.Cu")
     (at 139.0362 92.2784)
     (descr "Resistor, Axial_DIN0207 series, Axial, Vertical, pin pitch=5.08mm, 0.25W = 1/4W, length*diameter=6.3*2.5mm^2, http://cdn-reichelt.de/documents/datenblatt/B400/1_4W%23YAG.pdf")
@@
     (property "ki_keywords" "R res resistor")
     (attr through_hole)
-    (fp_text reference "R6" (at 2.54 -2.37) (layer "F.SilkS")
-        (effects (font (size 1 1) (thickness 0.15)))
-    )
-    (fp_text value "R" (at 0 0) (layer "F.Fab")
-        (effects (font (size 1 1) (thickness 0.15)))
-    )
-    (fp_text user "${REFERENCE}" (at 2.54 -2.37) (layer "F.Fab")
+    (fp_text reference "R9" (at 2.54 -2.37 180) (layer "F.SilkS")
+        (effects (font (size 1 1) (thickness 0.15)))
+    )
+    (fp_text value "R" (at 2.54 2.37 180) (layer "F.Fab")
+        (effects (font (size 1 1) (thickness 0.15)))
+    )
+    (fp_text user "${REFERENCE}" (at 2.54 -2.37 180) (layer "F.Fab")
         (effects (font (size 1 1) (thickness 0.15)))
     )
@@
     )
   )
-  (footprint "Resistor_THT:R_Axial_DIN0207_L6.3mm_D2.5mm_P5.08mm_Vertical" (layer "F.Cu")
+  (footprint "Library_Empreinte:R_Axial_DIN0207_L6.3mm_D2.5mm_P5.08mm_Vertical" (layer "F.Cu")
     (at 155.0128 53.4926)
     (descr "Resistor, Axial_DIN0207 series, Axial, Vertical, pin pitch=5.08mm, 0.25W = 1/4W, length*diameter=6.3*2.5mm^2, http://cdn-reichelt.de/documents/datenblatt/B400/1_4W%23YAG.pdf")
@@
     (property "ki_keywords" "R res resistor")
     (attr through_hole)
-    (fp_text reference "R2b1" (at 2.54 -2.37) (layer "F.SilkS")
-        (effects (font (size 1 1) (thickness 0.15)))
-    )
-    (fp_text value "R" (at 2.54 2.37) (layer "F.Fab")
-        (effects (font (size 1 1) (thickness 0.15)))
-    )
-    (fp_text user "${REFERENCE}" (at 2.54 -2.37) (layer "F.Fab")
+    (fp_text reference "R2b1" (at 2.54 -2.37 180) (layer "F.SilkS")
+        (effects (font (size 1 1) (thickness 0.15)))
+    )
+    (fp_text value "R" (at 2.54 2.37 180) (layer "F.Fab")
+        (effects (font (size 1 1) (thickness 0.15)))
+    )
+    (fp_text user "${REFERENCE}" (at 2.54 -2.37 180) (layer "F.Fab")
         (effects (font (size 1 1) (thickness 0.15)))
     )
@@
     )
   )
-  (footprint "Resistor_THT:R_Axial_DIN0207_L6.3mm_D2.5mm_P5.08mm_Vertical" (layer "F.Cu")
+  (footprint "Library_Empreinte:R_Axial_DIN0207_L6.3mm_D2.5mm_P5.08mm_Vertical" (layer "F.Cu")
     (at 126.0604 88.9038 90)
     (descr "Resistor, Axial_DIN0207 series, Axial, Vertical, pin pitch=5.08mm, 0.25W = 1/4W, length*diameter=6.3*2.5mm^2, http://cdn-reichelt.de/documents/datenblatt/B400/1_4W%23YAG.pdf")
@@
     (property "ki_keywords" "R res resistor")
     (attr through_hole)
-    (fp_text reference "R5" (at 2.54 -2.37 90) (layer "F.SilkS")
-        (effects (font (size 1 1) (thickness 0.15)))
-    )
-    (fp_text value "R" (at 2.54 2.37 90) (layer "F.Fab")
-        (effects (font (size 1 1) (thickness 0.15)))
-    )
-    (fp_text user "${REFERENCE}" (at 2.54 -2.37 90) (layer "F.Fab")
+    (fp_text reference "R5" (at 2.54 -2.37 270) (layer "F.SilkS")
+        (effects (font (size 1 1) (thickness 0.15)))
+    )
+    (fp_text value "R" (at 2.54 2.37 270) (layer "F.Fab")
+        (effects (font (size 1 1) (thickness 0.15)))
+    )
+    (fp_text user "${REFERENCE}" (at 2.54 -2.37 270) (layer "F.Fab")
         (effects (font (size 1 1) (thickness 0.15)))
     )
@@
     )
   )
-  (footprint "Resistor_THT:R_Axial_DIN0207_L6.3mm_D2.5mm_P5.08mm_Vertical" (layer "F.Cu")
+  (footprint "Library_Empreinte:R_Axial_DIN0207_L6.3mm_D2.5mm_P5.08mm_Vertical" (layer "F.Cu")
     (at 152.3966 57.6074)
     (descr "Resistor, Axial_DIN0207 series, Axial, Vertical, pin pitch=5.08mm, 0.25W = 1/4W, length*diameter=6.3*2.5mm^2, http://cdn-reichelt.de/documents/datenblatt/B400/1_4W%23YAG.pdf")
@@
     (property "ki_keywords" "R res resistor")
     (attr through_hole)
-    (fp_text reference "R7" (at 2.54 -2.37) (layer "F.SilkS")
-        (effects (font (size 1 1) (thickness 0.15)))
-    )
-    (fp_text value "R" (at 2.04 -1.38) (layer "F.Fab")
-        (effects (font (size 1 1) (thickness 0.15)))
-    )
-    (fp_text user "${REFERENCE}" (at 2.54 -2.37) (layer "F.Fab")
+    (fp_text reference "R7" (at 2.54 -2.37 180) (layer "F.SilkS")
+        (effects (font (size 1 1) (thickness 0.15)))
+    )
+    (fp_text value "R" (at 2.54 2.37 180) (layer "F.Fab")
+        (effects (font (size 1 1) (thickness 0.15)))
+    )
+    (fp_text user "${REFERENCE}" (at 2.54 -2.37 180) (layer "F.Fab")
         (effects (font (size 1 1) (thickness 0.15)))
     )
@@
     )
   )
-  (footprint "Resistor_THT:R_Axial_DIN0207_L6.3mm_D2.5mm_P5.08mm_Vertical" (layer "F.Cu")
+  (footprint "Library_Empreinte:R_Axial_DIN0207_L6.3mm_D2.5mm_P5.08mm_Vertical" (layer "F.Cu")
     (at 143.065 85.5 180)
     (descr "Resistor, Axial_DIN0207 series, Axial, Vertical, pin pitch=5.08mm, 0.25W = 1/4W, length*diameter=6.3*2.5mm^2, http://cdn-reichelt.de/documents/datenblatt/B400/1_4W%23YAG.pdf")
@@
     )
   )
-  (footprint "Resistor_THT:R_Axial_DIN0207_L6.3mm_D2.5mm_P5.08mm_Vertical" (layer "F.Cu")
+  (footprint "Library_Empreinte:R_Axial_DIN0207_L6.3mm_D2.5mm_P5.08mm_Vertical" (layer "F.Cu")
     (at 119.558 73.301 -90)
     (descr "Resistor, Axial_DIN0207 series, Axial, Vertical, pin pitch=5.08mm, 0.25W = 1/4W, length*diameter=6.3*2.5mm^2, http://cdn-reichelt.de/documents/datenblatt/B400/1_4W%23YAG.pdf")
@@
     (pad "" np_thru_hole circle locked (at 0 0) (size 3.2 3.2) (drill 3.2) (layers "*.Cu" "*.Mask"))
   )
-  (footprint "Resistor_THT:R_Axial_DIN0207_L6.3mm_D2.5mm_P5.08mm_Vertical" (layer "F.Cu")
+  (footprint "Library_Empreinte:R_Axial_DIN0207_L6.3mm_D2.5mm_P5.08mm_Vertical" (layer "F.Cu")
     (at 149.315 53.25 180)
     (descr "Resistor, Axial_DIN0207 series, Axial, Vertical, pin pitch=5.08mm, 0.25W = 1/4W, length*diameter=6.3*2.5mm^2, http://cdn-reichelt.de/documents/datenblatt/B400/1_4W%23YAG.pdf")
@@
     (property "ki_keywords" "R res resistor")
     (attr through_hole)
-    (fp_text reference "R8" (at 2.04 -6.12) (layer "F.SilkS")
-        (effects (font (size 1 1) (thickness 0.15)))
-    )
-    (fp_text value "R" (at 2.04 -1.38) (layer "F.Fab")
-        (effects (font (size 1 1) (thickness 0.15)))
-    )
-    (fp_text user "${REFERENCE}" (at 2.04 -6.12) (layer "F.Fab")
+    (fp_text reference "R8" (at 2.54 -2.37) (layer "F.SilkS")
+        (effects (font (size 1 1) (thickness 0.15)))
+    )
+    (fp_text value "R" (at 2.54 2.37) (layer "F.Fab")
+        (effects (font (size 1 1) (thickness 0.15)))
+    )
+    (fp_text user "${REFERENCE}" (at 2.54 -2.37) (layer "F.Fab")
         (effects (font (size 1 1) (thickness 0.15)))
     )
@@
   (gr_line (start 166.04 59.36) (end 168.58 61.9)
     (stroke (width 0.15) (type solid)) (layer "Edge.Cuts"))
-  (gr_line (start 99.873 102.921) (end 99.995471 47.422)
+  (gr_line (start 99.873 103.2512) (end 99.995471 47.422)
     (stroke (width 0.15) (type solid)) (layer "Edge.Cuts"))
   (gr_line (start 168.58 61.9) (end 168.58 96.19)
     (stroke (width 0.15) (type solid)) (layer "Edge.Cuts"))
-  (gr_line (start 166.04 102.921) (end 99.873 102.921)
+  (gr_line (start 166.04 103.2512) (end 99.873 103.2512)
     (stroke (width 0.15) (type solid)) (layer "Edge.Cuts"))
   (gr_line (start 101.905 45.644001) (end 163.5 45.75)
     (stroke (width 0.15) (type solid)) (layer "Edge.Cuts"))
-  (gr_line (start 168.58 96.19) (end 166.04 102.921)
+  (gr_line (start 168.58 96.19) (end 166.04 103.2512)
     (stroke (width 0.15) (type solid)) (layer "Edge.Cuts"))
   (gr_line (start 163.5 45.75) (end 166.04 47.803)
@@
         (xy 175 42.75)
         (xy 104.5 42.75)
-        (xy 104.75 102.75)
-        (xy 175.5 102.5)
+        (xy 104.7246 103.258)
+        (xy 175.1078 103.2004)
       )
     )
